File: heart.kicad_sch (KiCad schematic)
At the start: 20 parts, among them J1 Positive, J2 Negative, J3 Conn_01x19_Female, J4 Conn_01x19_Female, P1 USB_C_Plug_USB2.0, SW1 SW_DIP_x01, U1 BMD101, U2 TP4054, U3 RS3236, U5 RS8051

Commit message: 最终投板
Parts:
- removed P1: USB_C_Plug_USB2.0, Connector_USB:USB_C_Receptacle_XKB_U262-16XN-4BVC11, symbol Connector:USB_C_Plug_USB2.0
- added J5: USB_B_Mini, symbol Connector:USB_B_Mini
- added R5: 30 k, symbol Device:R
- added R6: 10 k, symbol Device:R
- BT1: value Battery_Cell -> (none); footprint Battery:BatteryHolder_Eagle_12BH611-GR -> (none)
- C1: value 0.1μF -> (none); footprint Capacitor_SMD:C_0805_2012Metric_Pad1.18x1.45mm_HandSolder -> (none)
- C2, C4: value 1μF -> (none); footprint Capacitor_SMD:C_0805_2012Metric_Pad1.18x1.45mm_HandSolder -> (none)
- C3: value 0.01μF -> (none); footprint Capacitor_SMD:C_0805_2012Metric_Pad1.18x1.45mm_HandSolder -> (none)
- D1: value LED -> (none); footprint LED_SMD:LED_0805_2012Metric_Pad1.15x1.40mm_HandSolder -> (none)
- J1: value Positive -> (none); footprint MountingHole:MountingHole_8.4mm_M8_Pad -> (none)
- J2: value Negative -> (none); footprint MountingHole:MountingHole_8.4mm_M8_Pad -> (none)
- J3, J4: value Conn_01x19_Female -> (none); footprint Connector_PinSocket_2.54mm:PinSocket_1x19_P2.54mm_Vertical -> (none)
- R1, R2: value 1K -> (none); footprint Resistor_SMD:R_0805_2012Metric_Pad1.20x1.40mm_HandSolder -> (none)
- R3: value MF52 -> (none); footprint Resistor_SMD:R_0805_2012Metric_Pad1.20x1.40mm_HandSolder -> (none)
- R4: value 1K -> 10 k; footprint Resistor_SMD:R_0805_2012Metric_Pad1.20x1.40mm_HandSolder -> (none)
- SW1: value SW_DIP_x01 -> (none); footprint Button_Switch_SMD:SW_DIP_SPSTx01_Slide_9.78x4.72mm_W8.61mm_P2.54mm -> (none)
- U1: value BMD101 -> (none); footprint Package_TO_SOT_SMD:BMD101 -> (none)
- U2: value TP4054 -> (none); footprint Package_TO_SOT_SMD:SOT-23-5 -> (none)
- U3: value RS3236 -> (none); footprint Package_TO_SOT_SMD:SOT-23-5 -> (none)
- U5: value RS8051 -> (none); footprint Package_TO_SOT_SMD:SOT-23-5 -> (none)
Connections:
- net ADC: no longer U5.1 (OUT)
- net BT+: no longer C2.1, U3.1 (IN)
- net GNDREF: now also R4.1, U5.2 (V-), J5.5 (GND), R6.2; no longer R4.2
- net VCC: now also U5.5 (V+), R5.2; no longer J3.2 (EN), R3.1
- net at C1.1, D1.2 (A), U2.4 (VCC): now also J5.1 (VBUS)
- net at SW1.2, U3.3 (EN): now also C2.1, U3.1 (IN)
- net at U5.4 (-IN): now also R3.2, R6.1
- removed net Temp: R3.2, R4.1, U5.3 (+IN)
- new net: R3.1, U5.1 (OUT)
- new net: R4.2, R5.1, U5.3 (+IN)
- no-connect marks 37 -> 35
Other:
- moved on the sheet: C2, J3, J4, R3, SW1, U5
